File: Hardware/CP2102 USB to Serial Breakout v12.brd (EAGLE design)
At the start: 34.3 x 25.4 mm, 18 parts, among them U1 CP2102, X1 USBPTH

Commit message: Version 1.3 files
Parts:
- added FRAME1: FRAME-LETTER, SparkFun-Aesthetics:CREATIVE_COMMONS
- added LOGO1: OSHW-LOGOS, SparkFun-Aesthetics:OSHW-LOGO-S
- added U$4: REVISION, SparkFun-Aesthetics:REVISION
- C1, C2: device SparkFun:0603 -> SparkFun-Capacitors:0603-CAP
- R1: device SparkFun:0603 -> SparkFun-Resistors:0603-RES
Other:
- board text added: "Aaron Weiss"
- board text added: "Toni Klopfenstein"
- board text added: "v13"
Changed lines of the file:
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@@
 <?xml version="1.0" encoding="utf-8"?>
 <!DOCTYPE eagle SYSTEM "eagle.dtd">
-<eagle version="6.4">
+<eagle version="6.5.0">
 <drawing>
 <settings>
@@
 <setting verticaltext="up"/>
 </settings>
-<grid distance="0.05" unitdist="inch" unit="inch" style="lines" multiple="1" display="yes" altdistance="0.005" altunitdist="inch" altunit="inch"/>
+<grid distance="0.025" unitdist="inch" unit="inch" style="lines" multiple="1" display="yes" altdistance="0.005" altunitdist="inch" altunit="inch"/>
 <layers>
 <layer number="1" name="Top" color="4" fill="1" visible="yes" active="yes"/>
@@
 <layer number="101" name="Patch_Top" color="12" fill="4" visible="no" active="yes"/>
 <layer number="102" name="Vscore" color="7" fill="1" visible="no" active="yes"/>
+<layer number="103" name="tMap" color="7" fill="1" visible="no" active="yes"/>
 <layer number="104" name="Name" color="7" fill="1" visible="no" active="yes"/>
+<layer number="105" name="tPlate" color="7" fill="1" visible="no" active="yes"/>
+<layer number="106" name="bPlate" color="7" fill="1" visible="no" active="yes"/>
+<layer number="107" name="Crop" color="7" fill="1" visible="no" active="yes"/>
 <layer number="116" name="Patch_BOT" color="9" fill="4" visible="no" active="yes"/>
 <layer number="121" name="_tsilk" color="7" fill="1" visible="no" active="yes"/>
 <layer number="122" name="_bsilk" color="7" fill="1" visible="no" active="yes"/>
+<layer number="125" name="_tNames" color="7" fill="1" visible="no" active="yes"/>
+<layer number="144" name="Drill_legend" color="7" fill="1" visible="no" active="yes"/>
 <layer number="151" name="HeatSink" color="7" fill="1" visible="no" active="yes"/>
+<layer number="199" name="Contour" color="7" fill="1" visible="yes" active="yes"/>
 <layer number="200" name="200bmp" color="1" fill="10" visible="no" active="no"/>
 <layer number="201" name="201bmp" color="2" fill="1" visible="no" active="no"/>
 <layer number="202" name="202bmp" color="3" fill="1" visible="no" active="no"/>
+<layer number="203" name="203bmp" color="4" fill="10" visible="no" active="yes"/>
+<layer number="204" name="204bmp" color="5" fill="10" visible="no" active="yes"/>
+<layer number="205" name="205bmp" color="6" fill="10" visible="no" active="yes"/>
+<layer number="206" name="206bmp" color="7" fill="10" visible="no" active="yes"/>
+<layer number="207" name="207bmp" color="8" fill="10" visible="no" active="yes"/>
+<layer number="208" name="208bmp" color="9" fill="10" visible="no" active="yes"/>
+<layer number="209" name="209bmp" color="7" fill="1" visible="no" active="yes"/>
+<layer number="210" name="210bmp" color="7" fill="1" visible="no" active="yes"/>
+<layer number="211" name="211bmp" color="7" fill="1" visible="no" active="yes"/>
+<layer number="212" name="212bmp" color="7" fill="1" visible="no" active="yes"/>
+<layer number="213" name="213bmp" color="7" fill="1" visible="no" active="yes"/>
+<layer number="214" name="214bmp" color="7" fill="1" visible="no" active="yes"/>
+<layer number="215" name="215bmp" color="7" fill="1" visible="no" active="yes"/>
+<layer number="216" name="216bmp" color="7" fill="1" visible="no" active="yes"/>
+<layer number="217" name="217bmp" color="18" fill="1" visible="no" active="no"/>
+<layer number="218" name="218bmp" color="19" fill="1" visible="no" active="no"/>
+<layer number="219" name="219bmp" color="20" fill="1" visible="no" active="no"/>
+<layer number="220" name="220bmp" color="21" fill="1" visible="no" active="no"/>
+<layer number="221" name="221bmp" color="22" fill="1" visible="no" active="no"/>
+<layer number="222" name="222bmp" color="23" fill="1" visible="no" active="no"/>
+<layer number="223" name="223bmp" color="24" fill="1" visible="no" active="no"/>
+<layer number="224" name="224bmp" color="25" fill="1" visible="no" active="no"/>
 <layer number="250" name="Descript" color="3" fill="1" visible="no" active="no"/>
 <layer number="251" name="SMDround" color="12" fill="11" visible="no" active="no"/>
@@
 <wire x1="34.29" y1="25.4" x2="0" y2="25.4" width="0.2032" layer="20"/>
 <wire x1="0" y1="25.4" x2="0" y2="0" width="0.2032" layer="20"/>
-<text x="27.305" y="15.875" size="1.4224" layer="21" ratio="15">3.3V</text>
-<text x="27.305" y="13.335" size="1.4224" layer="21" ratio="15">TXO</text>
-<text x="27.305" y="10.795" size="1.4224" layer="21" ratio="15">RXI</text>
-<text x="27.305" y="8.255" size="1.4224" layer="21" ratio="15">GND</text>
-<text x="23.495" y="23.241" size="1.778" layer="22" ratio="15" rot="MR0">VCC</text>
-<text x="23.495" y="20.701" size="1.778" layer="22" ratio="15" rot="MR0">DTR</text>
-<text x="23.495" y="18.161" size="1.778" layer="22" ratio="15" rot="MR0">DSR</text>
-<text x="23.495" y="15.621" size="1.778" layer="22" ratio="15" rot="MR0">RTS</text>
-<text x="23.495" y="13.081" size="1.778" layer="22" ratio="15" rot="MR0">CTS</text>
-<text x="23.495" y="10.541" size="1.778" layer="22" ratio="15" rot="MR0">RI</text>
-<text x="23.495" y="8.001" size="1.778" layer="22" ratio="15" rot="MR0">DCD</text>
-<text x="23.495" y="0.381" size="1.778" layer="22" ratio="15" rot="MR0">RST</text>
-<text x="23.495" y="5.461" size="1.778" layer="22" ratio="15" rot="MR0">SUSP1</text>
-<text x="23.495" y="2.921" size="1.778" layer="22" ratio="15" rot="MR0">SUSP2</text>
+<text x="27.305" y="15.875" size="1.4224" layer="21" font="vector" ratio="15">3.3V</text>
+<text x="27.305" y="13.335" size="1.4224" layer="21" font="vector" ratio="15">TXO</text>
+<text x="27.305" y="10.795" size="1.4224" layer="21" font="vector" ratio="15">RXI</text>
+<text x="27.305" y="8.255" size="1.4224" layer="21" font="vector" ratio="15">GND</text>
+<text x="23.495" y="23.241" size="1.778" layer="22" font="vector" ratio="15" rot="MR0">VCC</text>
+<text x="23.495" y="20.701" size="1.778" layer="22" font="vector" ratio="15" rot="MR0">DTR</text>
+<text x="23.495" y="18.161" size="1.778" layer="22" font="vector" ratio="15" rot="MR0">DSR</text>
+<text x="23.495" y="15.621" size="1.778" layer="22" font="vector" ratio="15" rot="MR0">RTS</text>
+<text x="23.495" y="13.081" size="1.778" layer="22" font="vector" ratio="15" rot="MR0">CTS</text>
+<text x="23.495" y="10.541" size="1.778" layer="22" font="vector" ratio="15" rot="MR0">RI</text>
+<text x="23.495" y="8.001" size="1.778" layer="22" font="vector" ratio="15" rot="MR0">DCD</text>
+<text x="23.495" y="0.381" size="1.778" layer="22" font="vector" ratio="15" rot="MR0">RST</text>
+<text x="23.495" y="5.461" size="1.778" layer="22" font="vector" ratio="15" rot="MR0">SUSP1</text>
+<text x="23.495" y="2.921" size="1.778" layer="22" font="vector" ratio="15" rot="MR0">SUSP2</text>
 <text x="13.97" y="17.78" size="1.4224" layer="21" font="vector" ratio="15">CP2102</text>
 <text x="12.954" y="16.002" size="1.4224" layer="21" font="vector" ratio="15">Breakout</text>
 <text x="16.002" y="1.016" size="1.4224" layer="21" font="vector" ratio="15">Power</text>
+<text x="25.4" y="-8.89" size="1.778" layer="51" font="vector" ratio="15">Aaron Weiss</text>
+<text x="25.4" y="-11.43" size="1.778" layer="51" font="vector" ratio="15">Toni Klopfenstein</text>
+<text x="33.655" y="21.59" size="1.016" layer="16" font="vector" ratio="25" rot="MR270">v13</text>
 </plain>
 <attributes>
@@
 <elements>
 <element name="U$1" library="SparkFun" package="SFE-NEW-WEBLOGO" value="LOGO-SFENEW" x="0.889" y="3.175" rot="MR90"/>
-<element name="C1" library="SparkFun" package="0603" value="1uF" x="16.51" y="6.35"/>
-<element name="C2" library="SparkFun" package="0603" value="0.1uF" x="19.05" y="20.32" rot="R180"/>
+<element name="C1" library="SparkFun-Capacitors" package="0603-CAP" value="1uF" x="16.51" y="6.35">
+<attribute name="PROD_ID" value="CAP-00868" x="16.51" y="6.35" size="1.778" layer="27" display="off"/>
+<attribute name="VALUE" value="1.0uF" x="16.51" y="6.35" size="1.778" layer="27" display="off"/>
+</element>
+<element name="C2" library="SparkFun-Capacitors" package="0603-CAP" value="0.1uF" x="19.05" y="20.32" rot="R180">
+<attribute name="PROD_ID" value="CAP-00810" x="19.05" y="20.32" size="1.778" layer="27" rot="R180" display="off"/>
+<attribute name="VALUE" value="0.1uF" x="19.05" y="20.32" size="1.778" layer="27" rot="R180" display="off"/>
+</element>
 <element name="C3" library="SparkFun" package="EIA3216" value="10uF" x="19.05" y="22.86"/>
 <element name="U1" library="SparkFun" package="MLP28" value="CP2102" x="19.05" y="12.7"/>
@@
 <element name="JP3" library="SparkFun" package="1X04" value="" x="33.02" y="16.51" rot="R270"/>
 <element name="JP4" library="SparkFun" package="1X10" value="M100.1" x="25.4" y="24.13" rot="R270"/>
-<element name="R1" library="SparkFun" package="0603" value="330" x="20.32" y="6.35" rot="R180"/>
+<element name="R1" library="SparkFun-Resistors" package="0603-RES" value="330" x="20.32" y="6.35" rot="R180">
+<attribute name="PROD_ID" value="RES-00818" x="20.32" y="6.35" size="1.778" layer="27" rot="R180" display="off"/>
+<attribute name="VALUE" value="330" x="20.32" y="6.35" size="1.778" layer="27" rot="R180" display="off"/>
+</element>
 <element name="LED1" library="SparkFun" package="LED-1206" value="Red" x="19.05" y="3.81"/>
 <element name="X1" library="SparkFun" package="USB-B-PTH" value="USBPTH" x="8.89" y="12.7"/>
@@
 <element name="U$8" library="SparkFun" package="STAND-OFF" value="STAND-OFF" x="30.48" y="22.86"/>
 <element name="U$9" library="SparkFun" package="STAND-OFF" value="STAND-OFF" x="30.48" y="2.54"/>
+<element name="FRAME1" library="SparkFun-Aesthetics" package="CREATIVE_COMMONS" value="FRAME-LETTER" x="-1.0684125" y="-8.89"/>
+<element name="U$4" library="SparkFun-Aesthetics" package="REVISION" value="REVISION" x="10.16" y="-11.43"/>
+<element name="LOGO1" library="SparkFun-Aesthetics" package="OSHW-LOGO-S" value="OSHW-LOGOS" x="29.21" y="12.7" rot="MR90"/>
 </elements>
 <signals>
