File: Hardware/CP2102 USB to Serial Breakout.brd (EAGLE design)
At the start: 34.3 x 25.4 mm, 21 parts, among them U1 CP2102, X1 USBPTH

Commit message: changed micro fiducial to regular
Parts:
- removed U$2, U$3: FIDUCIAL1X2, SparkFun:FIDUCIAL-1X2
- added FID1, FID2: FIDUCIAL1X2, SparkFun-Aesthetics:FIDUCIAL-1X2
