File: Hardware/CP2102 USB to Serial Breakout.sch (EAGLE design)
At the start: 21 parts, among them U1 CP2102, X1 USBPTH

Commit message: changed micro fiducial to regular
Parts:
- removed U$2, U$3: FIDUCIAL1X2, SparkFun:FIDUCIAL1X2
- added FID1, FID2: FIDUCIAL1X2, SparkFun-Aesthetics:FIDUCIAL1X2
Changed lines of the file:
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@@
 <part name="C3" library="SparkFun" deviceset="CAP_POL" device="1206" value="10uF"/>
 <part name="U1" library="SparkFun" deviceset="CP210X_USB_UART" device="" value="CP2102"/>
-<part name="U$2" library="SparkFun" deviceset="FIDUCIAL" device="1X2"/>
-<part name="U$3" library="SparkFun" deviceset="FIDUCIAL" device="1X2"/>
 <part name="GND1" library="SparkFun" deviceset="GND" device=""/>
 <part name="GND2" library="SparkFun" deviceset="GND" device=""/>
@@
 <part name="U$4" library="SparkFun-Aesthetics" deviceset="REVISION" device=""/>
 <part name="LOGO1" library="SparkFun-Aesthetics" deviceset="OSHW-LOGO" device="S"/>
+<part name="FID1" library="SparkFun-Aesthetics" deviceset="FIDUCIAL" device="1X2"/>
+<part name="FID2" library="SparkFun-Aesthetics" deviceset="FIDUCIAL" device="1X2"/>
 </parts>
 <sheets>
@@
 <instance part="C3" gate="G$1" x="53.34" y="104.14"/>
 <instance part="U1" gate="G$1" x="144.78" y="101.6"/>
-<instance part="U$2" gate="G$1" x="246.38" y="27.94"/>
-<instance part="U$3" gate="G$1" x="241.3" y="27.94"/>
 <instance part="GND1" gate="1" x="124.46" y="81.28"/>
 <instance part="GND2" gate="1" x="93.98" y="106.68"/>
@@
 <instance part="U$4" gate="G$1" x="149.352" y="6.858"/>
 <instance part="LOGO1" gate="G$1" x="132.08" y="12.7"/>
+<instance part="FID1" gate="G$1" x="241.3" y="27.94"/>
+<instance part="FID2" gate="G$1" x="246.38" y="27.94"/>
 </instances>
 <busses>
